File: suasPcbDesign.kicad_pcb (KiCad board)
At the start: 4 copper layers, 48 parts, among them U1 LMR51625DDC, U2 MCP3562RT-E/ST, U3 ESP32-S3-WROOM-1, U4 TLV77733PDBVR, X7R_Cap1 1uF, X7R_Cap2 1uF, X7R_Cap3 1uF, X7R_Cap4 0.1uF

Commit message: Merge and Organize Design
Parts:
- removed BT1: 60V, TerminalBlock_Phoenix:TerminalBlock_Phoenix_MKDS-1,5-2-5.08_1x02_P5.08mm_Horizontal
- removed L1: 12uH, suasPCBFootprints:L_Wurth_WE-MXGI-5030
- removed LCDDisplayConnector1: Conn_01x04, Connector_PinHeader_2.54mm:PinHeader_1x04_P2.54mm_Vertical
- removed R11: 0.005, Resistor_SMD:R_2512_6332Metric
- removed U1: LMR51625DDC, suasPCBFootprints:DDC0006A-MFG
- removed U2: MCP3562RT-E/ST, suasPCBFootprints:TSSOP20_ST_MCH
- removed U4: TLV77733PDBVR, suasPCBFootprints:TLV
- removed pmeter1: 23BR1KLFTR, suasPCBFootprints:RES3_23B_TTE
- added D1: LED_RGB, LED_SMD:LED_RGB_PLCC-6, F.Cu at (7.53, 45.1)
- added H1: BAT+, MountingHole:MountingHole_6.4mm_M6_Pad_Via, F.Cu at (6.67, 6.67)
- added H2: ESC-, MountingHole:MountingHole_6.4mm_M6, F.Cu at (6.67, 21.0)
- added H3: Bat-, MountingHole:MountingHole_6.4mm_M6_Pad_Via, F.Cu at (6.67, 35.4)
- added J1: SENSE_IB, Connector_Wire:SolderWire-0.25sqmm_1x02_P4.2mm_D0.65mm_OD1.7mm, F.Cu at (44.4, 51.6)
- added J2: USB_C_Receptacle_USB2.0_16P, Connector_USB:USB_C_Receptacle_GCT_USB4105-xx-A_16P_TopMnt_Horizontal, F.Cu at (36.4, 47.0)
- added R18: R, Resistor_SMD:R_0603_1608Metric_Pad0.98x0.95mm_HandSolder, F.Cu at (53.0, 48.0)
- added R19: 5.1k, Resistor_SMD:R_0805_2012Metric_Pad1.20x1.40mm_HandSolder, F.Cu at (1.88, 44.0)
- added R20: 5.1k, Resistor_SMD:R_0805_2012Metric_Pad1.20x1.40mm_HandSolder, F.Cu at (1.88, 47.0)
- added U5: USBLC6-2SC6, Package_TO_SOT_SMD:SOT-23-6, F.Cu at (6.83, 50.0)
- added Zener3: 3.3V, Diode_SMD:D_SOD-123, F.Cu at (58.1, 46.8)
- R16, R17: value 4.7k -> R; footprint Resistor_SMD:R_0402_1005Metric -> Resistor_SMD:R_0603_1608Metric_Pad0.98x0.95mm_HandSolder
- moved Loadcell1 175.7 mm to (28.3, 44.0), turned to 0 degrees
- moved R10 171.1 mm to (24.7, 53.1)
- moved R9 169.9 mm to (24.7, 51.4)
- moved R8 168.9 mm to (24.7, 49.6)
- moved R7 167.9 mm to (24.7, 47.9)
- moved R6 167.0 mm to (24.7, 46.1)
- moved R4 166.1 mm to (24.7, 44.4)
- moved R3 165.2 mm to (24.7, 42.6)
- moved U3 142.9 mm to (38.4, 27.8)
- moved R15 141.1 mm to (21.5, 53.0), turned to 0 degrees
- moved Cap11 140.1 mm to (43.7, 48.6), turned to 0 degrees
- moved R14 139.8 mm to (21.5, 50.5), turned to 0 degrees
- moved Cap12 139.4 mm to (46.5, 42.7), turned to 0 degrees
- moved R13 138.5 mm to (21.5, 48.0), turned to 0 degrees
- moved R12 137.7 mm to (21.5, 45.5), turned to 0 degrees
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Connections:
- net Net-(BT1-+) renamed /VIN
- net Net-(U2-CH0) renamed /SENSE_IB+
- net Net-(U2-CH1) renamed /SENSE_IB-
- net Net-(U2-CH2) renamed /SENSE_LC+
- net Net-(U2-CH3) renamed /SENSE_LC-
- net Net-(U3-IO1) renamed /SENSE_VB
- Cap_13 pad 2: GNDA -> GND
- Cout_Cap7 pad 1: Net-(Loadcell1-Pin_1) -> VDD
- Loadcell1 pad 1: Net-(Loadcell1-Pin_1) -> VDD
- R16 pad 1: Net-(Loadcell1-Pin_1) -> /IND_B
- R16 pad 2: Net-(LCDDisplayConnector1-Pin_2) -> Net-(D1-RA)
- R17 pad 1: Net-(LCDDisplayConnector1-Pin_1) -> /IND_G
- R17 pad 2: Net-(Loadcell1-Pin_1) -> Net-(D1-GA)
- R3 pad 2: Net-(Loadcell1-Pin_1) -> VDD
- R4 pad 1: Net-(Loadcell1-Pin_1) -> VDD
- U3 pad 12: Net-(LCDDisplayConnector1-Pin_1) -> /IND_R
- U3 pad 13: unconnected-(U3-USB_D--Pad13) -> /USB_D_N
- U3 pad 14: unconnected-(U3-USB_D+-Pad14) -> /USB_D_P
- U3 pad 2: Net-(Loadcell1-Pin_1) -> VDD
- U3 pad 6: unconnected-(U3-IO6-Pad6) -> /IND_B
- U3 pad 7: Net-(LCDDisplayConnector1-Pin_2) -> /IND_G
- Zener2 pad 1: Net-(Loadcell1-Pin_1) -> VDD

Commit message: Add indication lights
Parts:
- removed Cap10, Cap11, Cap12, Cap9, Cap_13, Cap_14, Cap_15, Cap_16, Cap_17: 0.1uF, Capacitor_SMD:C_0402_1005Metric
- removed Cap8, Cin_Cap6, Cout_Cap7: 1uF, Capacitor_SMD:C_0402_1005Metric
- removed Cboot_Cap4, X7R_Cap4: 0.1uF, Capacitor_SMD:C_0805_2012Metric
- removed Cout_Cap5: 47uF, Capacitor_SMD:C_1206_3216Metric
- removed D1: LED_RGB, LED_SMD:LED_RGB_PLCC-6
- removed H1: BAT+, MountingHole:MountingHole_6.4mm_M6_Pad_Via
- removed H2: ESC-, MountingHole:MountingHole_6.4mm_M6
- removed H3: Bat-, MountingHole:MountingHole_6.4mm_M6_Pad_Via
- removed J1: SENSE_IB, Connector_Wire:SolderWire-0.25sqmm_1x02_P4.2mm_D0.65mm_OD1.7mm
- removed J2: USB_C_Receptacle_USB2.0_16P, Connector_USB:USB_C_Receptacle_GCT_USB4105-xx-A_16P_TopMnt_Horizontal
- removed Loadcell1: Conn_01x04, Connector_PinHeader_2.54mm:PinHeader_1x04_P2.54mm_Vertical
- removed R1: 58k, Resistor_SMD:R_0402_1005Metric
- removed R10, R3, R4, R6, R7, R8, R9: 10, Resistor_SMD:R_0201_0603Metric
- removed R12, R13, R14, R15, R5: 100, Resistor_SMD:R_0603_1608Metric
- removed R16, R17, R18: R, Resistor_SMD:R_0603_1608Metric_Pad0.98x0.95mm_HandSolder
- removed R19, R20: 5.1k, Resistor_SMD:R_0805_2012Metric_Pad1.20x1.40mm_HandSolder
- removed R2: 1k, Resistor_SMD:R_0402_1005Metric
- removed Rfbb_R4: 10.2k, Resistor_SMD:R_0805_2012Metric
- removed Rfbt_R3: 47.5k, Resistor_SMD:R_0402_1005Metric
- removed U3: ESP32-S3-WROOM-1, RF_Module:ESP32-S3-WROOM-1
- removed U5: USBLC6-2SC6, Package_TO_SOT_SMD:SOT-23-6
- removed X7R_Cap1, X7R_Cap2, X7R_Cap3: 1uF, Capacitor_SMD:C_1206_3216Metric
- removed Zener1: 4.55V, Diode_SMD:D_SOD-123F
- removed Zener2, Zener3: 3.3V, Diode_SMD:D_SOD-123
