File: suasPcbDesign.kicad_pcb (KiCad board)
At the start: 4 copper layers, 71.6 x 100 mm, 100 parts, among them J1 SENSE_IB, J2 SPI CS, J4 SPI CTRL, J5 PWM CTRL, J6 JTAG Pinout, J7 USB_C_Receptacle_USB2.0_16P, M3x1 MountingHole_3.2mm_M3, M3x2 MountingHole_3.2mm_M3, M3x3 MountingHole_3.2mm_M3, M3x4 MountingHole_3.2mm_M3, SW1 SW_SPST, SW2 SW_SPST, SW3 SW_SPST, SW4 SW_SPST, SW5 SW_SPST, SW6 SW_SPST, SW7 SW_SPST, U1 74HC138, U2 LMR51625DDC, U3 MCP3562RT-E/ST, U4 MCP6486R, U5 TLV77733PDBVR, U6 LMV331, U7 ESP32-S3-WROOM-1, U8 LM66100DCK, U9 USBLC6-2SC6

Commit message: Add new comparator
Parts:
- R25: value 200R -> 300R

Commit message: Update part value for comparator
Parts:
- U6: value LMV331 -> MCP6541UT-E/OT
Changed lines of the file:
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@@
 			)
 		)
-		(property "Value" "LMV331"
+		(property "Value" "MCP6541UT-E/OT"
 			(at 0 2.9 90)
 			(layer "F.Fab")

Commit message: Fix diode position
Connections:
- BBCC1 pad 1: Net-(D9-K) -> /VIN
- BBCC2 pad 1: Net-(D9-K) -> /VIN
- BBCC3 pad 1: Net-(D9-K) -> /VIN
- BBCC4 pad 1: Net-(D9-K) -> /VIN
- D9 pad 1: Net-(D9-K) -> /VIN
- D9 pad 2: /VIN -> Net-(D9-A)
- H1 pad 1: /VIN -> Net-(D9-A)
- U2 pad 2: Net-(D9-K) -> /VIN
- U2 pad 3: Net-(D9-K) -> /VIN
Routing:
- net Net-(D9-A): track 0.00 -> 50.9 mm, vias 0 -> 1
- net /VIN: track 74.8 -> 56.4 mm
- added copper zone on F.Cu, net /VIN
- removed copper zone on F.Cu, net Net-(D9-K)
Changed lines of the file:
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@@
 			(layers "F.Cu" "F.Mask" "F.Paste")
 			(roundrect_rratio 0.25)
-			(net "Net-(D9-K)")
+			(net "/VIN")
 			(pintype "passive")
 		)
@@
 			(layers "F.Cu" "F.Mask" "F.Paste")
 			(roundrect_rratio 0.25)
-			(net "Net-(D9-K)")
+			(net "/VIN")
 			(pintype "passive")
 		)
@@
 			(layers "F.Cu" "F.Mask" "F.Paste")
 			(roundrect_rratio 0.25)
-			(net "Net-(D9-K)")
+			(net "/VIN")
 			(pintype "passive")
 		)
@@
 			(layers "*.Cu" "*.Mask")
 			(remove_unused_layers no)
-			(net "/VIN")
+			(net "Net-(D9-A)")
 			(pinfunction "1_1")
 			(pintype "input")
@@
 			(rect_delta 0.6 0)
 			(layers "F.Cu" "F.Mask" "F.Paste")
-			(net "Net-(D9-K)")
+			(net "/VIN")
 			(pinfunction "K_1")
 			(pintype "passive")
@@
 			(rect_delta 0.6 0)
 			(layers "F.Cu" "F.Mask" "F.Paste")
-			(net "/VIN")
+			(net "Net-(D9-A)")
 			(pinfunction "A_2")
 			(pintype "passive")
@@
 			(layers "F.Cu" "F.Mask" "F.Paste")
 			(roundrect_rratio 0.25)
-			(net "Net-(D9-K)")
+			(net "/VIN")
 			(pintype "passive")
 		)
@@
 			(layers "F.Cu" "F.Mask" "F.Paste")
 			(roundrect_rratio 0.25)
-			(net "Net-(D9-K)")
+			(net "/VIN")
 			(pinfunction "EN_2")
 			(pintype "input")
@@
 			(layers "F.Cu" "F.Mask" "F.Paste")
 			(roundrect_rratio 0.25)
-			(net "Net-(D9-K)")
+			(net "/VIN")
 			(pinfunction "VIN_3")
 			(pintype "power_in")
@@
 	)
 	(segment
-		(start 132.9 175.9)
-		(end 132.9 175)
-		(width 0.6)
-		(layer "F.Cu")
-		(net "/VIN")
-	)
-	(segment
 		(start 95 150.9125)
 		(end 95 177.9)
@@
 		(net "/VIN")
 	)
-	(segment
-		(start 132.9 175)
-		(end 131.3 173.4)
-		(width 0.6)
-		(layer "F.Cu")
-		(net "/VIN")
-	)
 	(via
 		(at 95 177.9)
@@
 	)
 	(via
-		(at 132.9 175.9)
+		(at 124.4 178)
 		(size 0.6)
 		(drill 0.3)
@@
 	)
 	(segment
-		(start 131.7 177.9)
-		(end 95 177.9)
-		(width 0.6)
-		(layer "In1.Cu")
-		(net "/VIN")
-	)
-	(segment
-		(start 94.7 177.9)
-		(end 93.1 179.5)
-		(width 0.6)
-		(layer "In1.Cu")
-		(net "/VIN")
-	)
-	(segment
-		(start 93.1 179.5)
-		(end 93.1 182.4)
-		(width 0.6)
-		(layer "In1.Cu")
-		(net "/VIN")
-	)
-	(segment
-		(start 132.9 175.9)
-		(end 132.9 176.7)
-		(width 0.6)
-		(layer "In1.Cu")
-		(net "/VIN")
-	)
-	(segment
-		(start 132.9 176.7)
-		(end 131.7 177.9)
-		(width 0.6)
+		(start 95 177.9)
+		(end 124.3 177.9)
+		(width 0.127)
 		(layer "In1.Cu")
 		(net "/VIN")
 	)
 	(segment
-		(start 95 177.9)
-		(end 94.7 177.9)
-		(width 0.6)
+		(start 124.3 177.9)
+		(end 124.4 178)
+		(width 0.127)
 		(layer "In1.Cu")
 		(net "/VIN")
@@
 		(net "Net-(D4-A)")
 	)
+	(segment
+		(start 134.3 180.7)
+		(end 134.3 176.4)
+		(width 0.6)
+		(layer "F.Cu")
+		(net "Net-(D9-A)")
+	)
+	(segment
+		(start 134.3 176.4)
+		(end 131.3 173.4)
+		(width 0.6)
+		(layer "F.Cu")
+		(net "Net-(D9-A)")
+	)
+	(via
+		(at 134.3 180.7)
+		(size 0.6)
+		(drill 0.3)
+		(layers "F.Cu" "B.Cu")
+		(net "Net-(D9-A)")
+	)
+	(segment
+		(start 101.948456 180.948456)
+		(end 104.948457 180.948456)
+		(width 0.6)
+		(layer "In1.Cu")
+		(net "Net-(D9-A)")
+	)
+	(segment
+		(start 104.948457 180.948456)
+		(end 105.196913 180.7)
+		(width 0.6)
+		(layer "In1.Cu")
+		(net "Net-(D9-A)")
+	)
+	(segment
+		(start 101.4 180.4)
+		(end 101.948456 180.948456)
+		(width 0.6)
+		(layer "In1.Cu")
+		(net "Net-(D9-A)")
+	)
+	(segment
+		(start 95.1 180.4)
+		(end 101.4 180.4)
+		(width 0.6)
+		(layer "In1.Cu")
+		(net "Net-(D9-A)")
+	)
+	(segment
+		(start 93.1 182.4)
+		(end 95.1 180.4)
+		(width 0.6)
+		(layer "In1.Cu")
+		(net "Net-(D9-A)")
+	)
+	(segment
+		(start 105.196913 180.7)
+		(end 134.3 180.7)
+		(width 0.6)
+		(layer "In1.Cu")
+		(net "Net-(D9-A)")
+	)
 	(zone
 		(net "VDD")
@@
 	)
 	(zone
-		(net "Net-(D9-K)")
+		(net "/VIN")
 		(layer "F.Cu")
 		(hatch edge 0.5)
